Commit message: Fix FR20 inertial origins with best guesses

File: fairino_description/urdf/fairino20_v6/fairino20_v6.description.xacro (robot description, xacro)
@@ -47,5 +47,5 @@
     <link name="${prefix}shoulder_link">
       <inertial>
-        <origin xyz="-0.00019 -0.03657 0.00568" rpy="0 0 0" />
+        <origin xyz="-0.00019 -0.03657 0.215" rpy="0 0 0" />
         <mass value="20.79" />
         <inertia ixx="0.11681303" ixy="0.000010684" ixz="0.00015198" iyy="0.09147711"
@@ -81,5 +81,5 @@
     <link name="${prefix}upperarm_link">
       <inertial>
-        <origin xyz="0.60525 0.00006 0.20294" rpy="0 0 0" />
+        <origin xyz="-0.60525 0.00006 0.20294" rpy="0 0 0" />
         <mass value="42.84" />
         <inertia ixx="0.21509702" ixy="0.00193218" ixz="0.11070934" iyy="8.34192406"
@@ -115,5 +115,5 @@
     <link name="${prefix}forearm_link">
       <inertial>
-        <origin xyz="0.26284 0.00022 0.04308" rpy="0 0 0" />
+        <origin xyz="-0.26284 0.00022 0.04308" rpy="0 0 0" />
         <mass value="9.88" />
         <inertia ixx="0.03036772" ixy="0.00023857" ixz="0.00627398" iyy="0.86016899"
@@ -148,5 +148,5 @@
     <link name="${prefix}wrist1_link">
       <inertial>
-        <origin xyz="0.00023 -0.00228 0.01842" rpy="0 0 0" />
+        <origin xyz="0.00023 -0.00228 0.166" rpy="0 0 0" />
         <mass value="4.64" />
         <inertia ixx="0.00933772" ixy="0.00003325" ixz="0.00005007" iyy="0.00926897"
@@ -181,5 +181,5 @@
     <link name="${prefix}wrist2_link">
       <inertial>
-        <origin xyz="-0.00023 0.00228 0.01842" rpy="0 0 0" />
+        <origin xyz="-0.00023 0.00228 0.138" rpy="0 0 0" />
         <mass value="4.64" />
         <inertia ixx="0.00933772" ixy="0.00003325" ixz="-0.00005007" iyy="0.00926897"
@@ -214,5 +214,5 @@
     <link name="${prefix}wrist3_link">
       <inertial>
-        <origin xyz="-0.00211 -0.00196 -0.02038" rpy="0 0 0" />
+        <origin xyz="-0.00211 -0.00196 0.102" rpy="0 0 0" />
         <mass value="0.6" />
         <inertia ixx="0.00071709" ixy="0.00000175" ixz="0.00000555" iyy="0.00071408"

Commit message: Fix FR20 joint effort limits with torque calculations based on link and payload mass

File: fairino_description/urdf/fairino20_v6/fairino20_v6.description.xacro (robot description, xacro)
@@ -39,5 +39,5 @@
       <child link="${prefix}shoulder_link" />
       <axis xyz="0 0 1" />
-      <limit lower="-3.0543" upper="3.0543" effort="150" velocity="3.15" />
+      <limit lower="-3.0543" upper="3.0543" effort="1100" velocity="3.15" />
       <calibration rising="0" falling="0" />
       <dynamics damping="0" friction="0" />
@@ -73,5 +73,5 @@
       <child link="${prefix}upperarm_link" />
       <axis xyz="0 0 1" />
-      <limit lower="-4.6251" upper="1.4835" effort="150" velocity="3.15" />
+      <limit lower="-4.6251" upper="1.4835" effort="1100" velocity="3.15" />
       <calibration rising="0" falling="0" />
       <dynamics damping="0" friction="0" />
@@ -107,5 +107,5 @@
       <child link="${prefix}forearm_link" />
       <axis xyz="0 0 1" />
-      <limit lower="-2.8274" upper="2.8274" effort="150" velocity="3.15" />
+      <limit lower="-2.8274" upper="2.8274" effort="350" velocity="3.15" />
       <calibration rising="0" falling="0" />
       <dynamics damping="0" friction="0" />
@@ -140,5 +140,5 @@
       <child link="${prefix}wrist1_link" />
       <axis xyz="0 0 1" />
-      <limit lower="-4.6251" upper="1.4835" effort="28" velocity="3.2" />
+      <limit lower="-4.6251" upper="1.4835" effort="60" velocity="3.2" />
       <calibration rising="0" falling="0" />
       <dynamics damping="0" friction="0" />
@@ -173,5 +173,5 @@
       <child link="${prefix}wrist2_link" />
       <axis xyz="0 0 1" />
-      <limit lower="-3.0543" upper="3.0543" effort="28" velocity="3.2" />
+      <limit lower="-3.0543" upper="3.0543" effort="60" velocity="3.2" />
       <calibration rising="0" falling="0" />
       <dynamics damping="0" friction="0" />
@@ -206,5 +206,5 @@
       <child link="${prefix}wrist3_link" />
       <axis xyz="0 0 1" />
-      <limit lower="-3.0543" upper="3.0543" effort="28" velocity="3.2" />
+      <limit lower="-3.0543" upper="3.0543" effort="60" velocity="3.2" />
       <calibration rising="0" falling="0" />
       <dynamics damping="0" friction="0" />
