Commit message: Add FR10 collision meshes from CoACD

File: fairino_description/urdf/fairino10_v6/fairino10_v6.description.xacro (robot description, xacro)
@@ -29,5 +29,5 @@
         <origin xyz="0 0 0" rpy="0 0 0" />
         <geometry>
-          <mesh filename="package://fairino_description/meshes/fairino10_v6/visual/base_link.stl" />
+          <mesh filename="package://fairino_description/meshes/fairino10_v6/collision/base_link_collision.stl" />
         </geometry>
       </collision>
@@ -61,5 +61,5 @@
         <origin xyz="0 0 0" rpy="0 0 0" />
         <geometry>
-          <mesh filename="package://fairino_description/meshes/fairino10_v6/visual/shoulder_link.stl" />
+          <mesh filename="package://fairino_description/meshes/fairino10_v6/collision/shoulder_link_collision.stl" />
         </geometry>
       </collision>
@@ -93,5 +93,5 @@
         <origin xyz="0 0 0" rpy="0 0 0" />
         <geometry>
-          <mesh filename="package://fairino_description/meshes/fairino10_v6/visual/upperarm_link.stl" />
+          <mesh filename="package://fairino_description/meshes/fairino10_v6/collision/upperarm_link_collision.stl" />
         </geometry>
       </collision>
@@ -125,5 +125,5 @@
         <origin xyz="0 0 0" rpy="0 0 0" />
         <geometry>
-          <mesh filename="package://fairino_description/meshes/fairino10_v6/visual/forearm_link.stl" />
+          <mesh filename="package://fairino_description/meshes/fairino10_v6/collision/forearm_link_collision.stl" />
         </geometry>
       </collision>
@@ -157,5 +157,5 @@
         <origin xyz="0 0 0" rpy="0 0 0" />
         <geometry>
-          <mesh filename="package://fairino_description/meshes/fairino10_v6/visual/wrist1_link.stl" />
+          <mesh filename="package://fairino_description/meshes/fairino10_v6/collision/wrist1_link_collision.stl" />
         </geometry>
       </collision>
@@ -189,5 +189,5 @@
         <origin xyz="0 0 0" rpy="0 0 0" />
         <geometry>
-          <mesh filename="package://fairino_description/meshes/fairino10_v6/visual/wrist2_link.stl" />
+          <mesh filename="package://fairino_description/meshes/fairino10_v6/collision/wrist2_link_collision.stl" />
         </geometry>
       </collision>
@@ -221,5 +221,5 @@
         <origin xyz="0 0 0" rpy="0 0 0" />
         <geometry>
-          <mesh filename="package://fairino_description/meshes/fairino10_v6/visual/wrist3_link.stl" />
+          <mesh filename="package://fairino_description/meshes/fairino10_v6/collision/wrist3_link_collision.stl" />
         </geometry>
       </collision>

Commit message: Fix FR10 inertial origins with best guesses

File: fairino_description/urdf/fairino10_v6/fairino10_v6.description.xacro (robot description, xacro)
@@ -46,5 +46,5 @@
     <link name="${prefix}shoulder_link">
       <inertial>
-        <origin xyz="-0.0001 -0.02612 0.00404" rpy="0 0 0" />
+        <origin xyz="-0.0001 -0.02612 0.18" rpy="0 0 0" />
         <mass value="11.97" />
         <inertia ixx="0.04607471" ixy="-0.00001041" ixz="-0.00009371" iyy="0.03493881"
@@ -78,5 +78,5 @@
     <link name="${prefix}upperarm_link">
       <inertial>
-        <origin xyz="0.48027 0.00001 0.16468" rpy="0 0 0" />
+        <origin xyz="-0.48027 0.00001 0.16468" rpy="0 0 0" />
         <mass value="19.59" />
         <inertia ixx="0.0649166" ixy="0.00054242" ixz="-0.02821532" iyy="1.81964752"
@@ -110,5 +110,5 @@
     <link name="${prefix}forearm_link">
       <inertial>
-        <origin xyz="0.21122 0.00011 0.05421" rpy="0 0 0" />
+        <origin xyz="-0.21122 0.00011 0.05421" rpy="0 0 0" />
         <mass value="3.7" />
         <inertia ixx="0.00642901" ixy="0.00004731" ixz="0.00070041" iyy="0.20273064"
@@ -142,5 +142,5 @@
     <link name="${prefix}wrist1_link">
       <inertial>
-        <origin xyz="0.00012 -0.003 0.01218" rpy="0 0 0" />
+        <origin xyz="0.00012 -0.003 0.159" rpy="0 0 0" />
         <mass value="1.69" />
         <inertia ixx="0.00248058" ixy="0.00001495" ixz="0.00002165" iyy="0.00239729"
@@ -174,5 +174,5 @@
     <link name="${prefix}wrist2_link">
       <inertial>
-        <origin xyz="-0.00012 0.003 0.01218" rpy="0 0 0" />
+        <origin xyz="-0.00012 0.003 0.114" rpy="0 0 0" />
         <mass value="1.69" />
         <inertia ixx="0.00248058" ixy="0.00001495" ixz="-0.00002165" iyy="0.00239729"
@@ -206,5 +206,5 @@
     <link name="${prefix}wrist3_link">
       <inertial>
-        <origin xyz="0.00124 0.00085 -0.02034" rpy="0 0 0" />
+        <origin xyz="0.00124 0.00085 0.084" rpy="0 0 0" />
         <mass value="0.35" />
         <inertia ixx="0.00023661" ixy="-0.00000085" ixz="0.00000092" iyy="0.00023501"

Commit message: Fix FR10 and FR20 joint effort limits with calculations based on link and payload mass, and payload offset curves

File: fairino_description/urdf/fairino10_v6/fairino10_v6.description.xacro (robot description, xacro)
@@ -38,5 +38,5 @@
       <child link="${prefix}shoulder_link" />
       <axis xyz="0 0 1" />
-      <limit lower="-3.0543" upper="3.0543" effort="150" velocity="3.15" />
+      <limit lower="-3.0543" upper="3.0543" effort="400" velocity="3.15" />
       <calibration rising="0" falling="0" />
       <dynamics damping="0" friction="0" />
@@ -70,5 +70,5 @@
       <child link="${prefix}upperarm_link" />
       <axis xyz="0 0 1" />
-      <limit lower="-4.6251" upper="1.4835" effort="150" velocity="3.15" />
+      <limit lower="-4.6251" upper="1.4835" effort="400" velocity="3.15" />
       <calibration rising="0" falling="0" />
       <dynamics damping="0" friction="0" />
@@ -134,5 +134,5 @@
       <child link="${prefix}wrist1_link" />
       <axis xyz="0 0 1" />
-      <limit lower="-4.6251" upper="1.4835" effort="28" velocity="3.2" />
+      <limit lower="-4.6251" upper="1.4835" effort="50" velocity="3.2" />
       <calibration rising="0" falling="0" />
       <dynamics damping="0" friction="0" />
@@ -166,5 +166,5 @@
       <child link="${prefix}wrist2_link" />
       <axis xyz="0 0 1" />
-      <limit lower="-3.0543" upper="3.0543" effort="28" velocity="3.2" />
+      <limit lower="-3.0543" upper="3.0543" effort="50" velocity="3.2" />
       <calibration rising="0" falling="0" />
       <dynamics damping="0" friction="0" />
@@ -198,5 +198,5 @@
       <child link="${prefix}wrist3_link" />
       <axis xyz="0 0 1" />
-      <limit lower="-3.0543" upper="3.0543" effort="28" velocity="3.2" />
+      <limit lower="-3.0543" upper="3.0543" effort="50" velocity="3.2" />
       <calibration rising="0" falling="0" />
       <dynamics damping="0" friction="0" />

File: fairino_description/urdf/fairino20_v6/fairino20_v6.description.xacro (robot description, xacro)
@@ -107,5 +107,5 @@
       <child link="${prefix}forearm_link" />
       <axis xyz="0 0 1" />
-      <limit lower="-2.8274" upper="2.8274" effort="350" velocity="3.15" />
+      <limit lower="-2.8274" upper="2.8274" effort="400" velocity="3.15" />
       <calibration rising="0" falling="0" />
       <dynamics damping="0" friction="0" />
@@ -140,5 +140,5 @@
       <child link="${prefix}wrist1_link" />
       <axis xyz="0 0 1" />
-      <limit lower="-4.6251" upper="1.4835" effort="60" velocity="3.2" />
+      <limit lower="-4.6251" upper="1.4835" effort="100" velocity="3.2" />
       <calibration rising="0" falling="0" />
       <dynamics damping="0" friction="0" />
@@ -173,5 +173,5 @@
       <child link="${prefix}wrist2_link" />
       <axis xyz="0 0 1" />
-      <limit lower="-3.0543" upper="3.0543" effort="60" velocity="3.2" />
+      <limit lower="-3.0543" upper="3.0543" effort="100" velocity="3.2" />
       <calibration rising="0" falling="0" />
       <dynamics damping="0" friction="0" />
@@ -206,5 +206,5 @@
       <child link="${prefix}wrist3_link" />
       <axis xyz="0 0 1" />
-      <limit lower="-3.0543" upper="3.0543" effort="60" velocity="3.2" />
+      <limit lower="-3.0543" upper="3.0543" effort="100" velocity="3.2" />
       <calibration rising="0" falling="0" />
       <dynamics damping="0" friction="0" />

Commit message: Update FR10 and FR20 joint effort limits again, this time based on fairino_gazebo repo

File: fairino_description/urdf/fairino10_v6/fairino10_v6.description.xacro (robot description, xacro)
@@ -38,5 +38,5 @@
       <child link="${prefix}shoulder_link" />
       <axis xyz="0 0 1" />
-      <limit lower="-3.0543" upper="3.0543" effort="400" velocity="3.15" />
+      <limit lower="-3.0543" upper="3.0543" effort="635" velocity="3.15" />
       <calibration rising="0" falling="0" />
       <dynamics damping="0" friction="0" />
@@ -70,5 +70,5 @@
       <child link="${prefix}upperarm_link" />
       <axis xyz="0 0 1" />
-      <limit lower="-4.6251" upper="1.4835" effort="400" velocity="3.15" />
+      <limit lower="-4.6251" upper="1.4835" effort="635" velocity="3.15" />
       <calibration rising="0" falling="0" />
       <dynamics damping="0" friction="0" />
@@ -102,5 +102,5 @@
       <child link="${prefix}forearm_link" />
       <axis xyz="0 0 1" />
-      <limit lower="-2.8274" upper="2.8274" effort="150" velocity="3.15" />
+      <limit lower="-2.8274" upper="2.8274" effort="332" velocity="3.15" />
       <calibration rising="0" falling="0" />
       <dynamics damping="0" friction="0" />
@@ -134,5 +134,5 @@
       <child link="${prefix}wrist1_link" />
       <axis xyz="0 0 1" />
-      <limit lower="-4.6251" upper="1.4835" effort="50" velocity="3.2" />
+      <limit lower="-4.6251" upper="1.4835" effort="110" velocity="3.2" />
       <calibration rising="0" falling="0" />
       <dynamics damping="0" friction="0" />
@@ -166,5 +166,5 @@
       <child link="${prefix}wrist2_link" />
       <axis xyz="0 0 1" />
-      <limit lower="-3.0543" upper="3.0543" effort="50" velocity="3.2" />
+      <limit lower="-3.0543" upper="3.0543" effort="110" velocity="3.2" />
       <calibration rising="0" falling="0" />
       <dynamics damping="0" friction="0" />
@@ -198,5 +198,5 @@
       <child link="${prefix}wrist3_link" />
       <axis xyz="0 0 1" />
-      <limit lower="-3.0543" upper="3.0543" effort="50" velocity="3.2" />
+      <limit lower="-3.0543" upper="3.0543" effort="110" velocity="3.2" />
       <calibration rising="0" falling="0" />
       <dynamics damping="0" friction="0" />

File: fairino_description/urdf/fairino20_v6/fairino20_v6.description.xacro (robot description, xacro)
@@ -39,5 +39,5 @@
       <child link="${prefix}shoulder_link" />
       <axis xyz="0 0 1" />
-      <limit lower="-3.0543" upper="3.0543" effort="1100" velocity="3.15" />
+      <limit lower="-3.0543" upper="3.0543" effort="1400" velocity="3.15" />
       <calibration rising="0" falling="0" />
       <dynamics damping="0" friction="0" />
@@ -73,5 +73,5 @@
       <child link="${prefix}upperarm_link" />
       <axis xyz="0 0 1" />
-      <limit lower="-4.6251" upper="1.4835" effort="1100" velocity="3.15" />
+      <limit lower="-4.6251" upper="1.4835" effort="1400" velocity="3.15" />
       <calibration rising="0" falling="0" />
       <dynamics damping="0" friction="0" />
@@ -107,5 +107,5 @@
       <child link="${prefix}forearm_link" />
       <axis xyz="0 0 1" />
-      <limit lower="-2.8274" upper="2.8274" effort="400" velocity="3.15" />
+      <limit lower="-2.8274" upper="2.8274" effort="635" velocity="3.15" />
       <calibration rising="0" falling="0" />
       <dynamics damping="0" friction="0" />
@@ -140,5 +140,5 @@
       <child link="${prefix}wrist1_link" />
       <axis xyz="0 0 1" />
-      <limit lower="-4.6251" upper="1.4835" effort="100" velocity="3.2" />
+      <limit lower="-4.6251" upper="1.4835" effort="332" velocity="3.2" />
       <calibration rising="0" falling="0" />
       <dynamics damping="0" friction="0" />
@@ -173,5 +173,5 @@
       <child link="${prefix}wrist2_link" />
       <axis xyz="0 0 1" />
-      <limit lower="-3.0543" upper="3.0543" effort="100" velocity="3.2" />
+      <limit lower="-3.0543" upper="3.0543" effort="332" velocity="3.2" />
       <calibration rising="0" falling="0" />
       <dynamics damping="0" friction="0" />
@@ -206,5 +206,5 @@
       <child link="${prefix}wrist3_link" />
       <axis xyz="0 0 1" />
-      <limit lower="-3.0543" upper="3.0543" effort="100" velocity="3.2" />
+      <limit lower="-3.0543" upper="3.0543" effort="332" velocity="3.2" />
       <calibration rising="0" falling="0" />
       <dynamics damping="0" friction="0" />
