Commit message: Regenerate FR20 MoveIt config

File: fairino20_v6_moveit2_config/config/fairino20_v6_robot.urdf.xacro (robot description, xacro)
@@ -1,9 +1,5 @@
 <?xml version="1.0"?>
 <robot xmlns:xacro="http://www.ros.org/wiki/xacro" name="fairino20_v6_robot">
-    <xacro:arg name="initial_positions_file" default="initial_positions.yaml" />
-    <!-- Import fairino20_v6_robot urdf file -->
-    <xacro:include filename="$(find fairino_description)/urdf/fairino20_v6.urdf" />
-    <!-- Import control_xacro -->
-    <xacro:include filename="fairino20_v6_robot.ros2_control.xacro" />
-    <xacro:fairino20_v6_robot_ros2_control name="FakeSystem" initial_positions_file="$(arg initial_positions_file)"/>
+  <!-- Import fairino20_v6_robot urdf file -->
+  <xacro:include filename="$(find fairino_description)/urdf/fairino20_v6/fairino20_v6.urdf.xacro" />
 </robot>

File: fairino_description/urdf/fairino20_v6/fairino20_v6.ros2_control.xacro (robot description, xacro)
@@ -2,5 +2,5 @@
 <!-- This URDF was artisanally crafted by Jacob Beck (jbeck@spaceroboticsworkers.com) -->
 <robot xmlns:xacro="http://wiki.ros.org/xacro">
-  <xacro:macro name="fairino20_v6_control" params="prefix mode">
+  <xacro:macro name="fairino20_v6_ros2_control" params="prefix mode">
     <ros2_control name="${prefix}fairino20_v6_system" type="system">
       <!-- Load appropriate hardware plugin -->
@@ -13,6 +13,5 @@
         </xacro:if>
         <xacro:if value="${mode == 'real'}">
-          <!-- TODO: Create control plugin -->
-          <plugin>fairino_custom_driver/FairinoDriver</plugin>
+          <plugin>fairino_hardware/FairinoHardwareInterface</plugin>
         </xacro:if>
       </hardware>

File: fairino_description/urdf/fairino20_v6/fairino20_v6.urdf.xacro (robot description, xacro)
@@ -12,5 +12,5 @@
     default="$(find fairino20_v6_moveit2_config)/config/ros2_controllers.yaml" />
   <!-- Include required macros -->
-  <xacro:include filename="$(find fairino_description)/urdf/fairino20_v6/fairino20_v6.control.xacro" />
+  <xacro:include filename="$(find fairino_description)/urdf/fairino20_v6/fairino20_v6.ros2_control.xacro" />
   <xacro:include
     filename="$(find fairino_description)/urdf/fairino20_v6/fairino20_v6.description.xacro" />
@@ -21,5 +21,5 @@
     <origin xyz="$(arg xyz)" rpy="$(arg rpy)" />
   </xacro:fairino20_v6_description>
-  <xacro:fairino20_v6_control prefix="$(arg prefix)" mode="$(arg mode)" />
+  <xacro:fairino20_v6_ros2_control prefix="$(arg prefix)" mode="$(arg mode)" />
   <xacro:property name="mode" value="$(arg mode)" /> <!-- Get arg as property for evaluation -->
   <xacro:if value="${mode == 'gazebo'}">
